Commit message: Codex correcting issue with steering bounds and corrected command timeouts.

File: src/swervebot_description/description/swervebot_properties.xacro (robot description, xacro)
@@ -31,6 +31,6 @@
   <!-- Actuator Limits -->
   <!--  (In radians)   -->
-  <xacro:property name="actuator_pos_min" value="-3.14159"/>
-  <xacro:property name="actuator_pos_max" value="-3.14159"/>
+  <xacro:property name="actuator_pos_min" value="-1.5708"/>
+  <xacro:property name="actuator_pos_max" value="1.5708"/>
   <!-- Material & Visual Properties -->
   <xacro:property name="wheel_color" value="0.1 0.1 0.1 1.0"/>

Commit message: [200~refactor: Generalize swerve kinematics to support arbitrary N-module layouts
- Replaced hardcoded rectangular geometry scalars with equal-length arrays
- Added parameter handling for module_x, module_y, wheel_radii, wheel_offsets,
  steering_continuous, steering_min, steering_max, and steering_velocity_limits
- Validated N>=3 module configurations and added array size matching checks in on_configure
- Verified fix with 159 passing unit/integration tests and active simulation joint states

File: src/swervebot_description/description/swervebot_properties.xacro (robot description, xacro)
@@ -28,4 +28,19 @@
   <!-- Chassis Ground Clearance -->
   <xacro:property name="chassis_ground_clearance" value="${wheel_radius - actuator_offset_z - wheel_offset_z - chassis_height/2}" />
+  <!-- Lidar Properties -->
+  <xacro:property name="lidar_radius" value="0.03"/>
+  <xacro:property name="lidar_height" value="0.04"/>
+  <xacro:property name="lidar_mass" value="0.1"/>
+  <xacro:property name="lidar_samples" value="500"/>
+  <xacro:property name="lidar_angle_res" value="1"/>
+  <xacro:property name="lidar_min_angle" value="-3.14159"/>
+  <xacro:property name="lidar_max_angle" value="3.14159"/>
+  <xacro:property name="lidar_min_range" value="0.05"/>
+  <xacro:property name="lidar_max_range" value="12.0"/>
+  <xacro:property name="lidar_range_res" value="0.01"/>
+  <!-- Lidar Position -->
+  <xacro:property name="lidar_x" value="0.15"/>
+  <xacro:property name="lidar_y" value="0.0"/>
+  <xacro:property name="lidar_z" value="${chassis_ground_clearance + chassis_height + (lidar_height / 2)}"/>
   <!--   ~ LIMITS ~    -->
   <!-- Actuator Limits -->
@@ -42,4 +57,5 @@
   <xacro:property name="chassis_color" value="0.7 0.7 0.7 1.0"/>
   <xacro:property name="actuator_color" value="1 0.5 0.5 1.0" />
+  <xacro:property name="lidar_color" value="0.9 0.9 0.9 1.0" />
   <!-- ============================================ -->
   <!--                 Module Names                 -->
