Commit message: Added teleop package for control input mapping.

File: src/swervebot_description/description/swervebot.urdf.xacro (robot description, xacro)
@@ -8,4 +8,5 @@
     <xacro:arg name="use_sim" default="false"/>
     <xacro:arg name="use_mock_hardware" default="false"/>
+    <xacro:arg name="controller_config" default="$(find swervebot_controllers)/config/controllers.yaml"/>
     <!-- Execute/Instantiate the macros -->
     <xacro:swervebot_base />
@@ -14,4 +15,5 @@
         use_mock_hardware="$(arg use_mock_hardware)"
         use_sim="$(arg use_sim)"
+        controller_config="$(arg controller_config)"
     />
 </robot>

File: src/swervebot_description/description/swervebot_actuator.xacro (robot description, xacro)
@@ -5,9 +5,12 @@
     <xacro:include filename="$(find swervebot_description)/description/inertia.xacro" />
     <xacro:macro name="swervebot_actuator" params="name x y z parent_link">
-        <joint name="${name}_joint" type="continuous">
+        <joint name="${name}_joint" type="revolute">
             <parent link="${parent_link}" />
             <child link="${name}" />
             <origin xyz="${x} ${y} ${z}" rpy="0 0 0" />
             <axis xyz="0 0 1" />
+            <!-- Mechanical travel must agree with the ros2_control command bounds. -->
+            <limit lower="${actuator_pos_min}" upper="${actuator_pos_max}"
+                   velocity="${actuator_velocity_limit}" effort="${actuator_effort_limit}"/>
         </joint>
         <link name="${name}">

File: src/swervebot_description/description/swervebot_properties.xacro (robot description, xacro)
@@ -27,10 +27,15 @@
   <xacro:property name="actuator_offset_z" value="-0.025"/>
   <!-- Chassis Ground Clearance -->
-  <xacro:property name="chassis_ground_clearance" value="0.1" />
+  <xacro:property name="chassis_ground_clearance" value="${wheel_radius - actuator_offset_z - wheel_offset_z - chassis_height/2}" />
   <!--   ~ LIMITS ~    -->
   <!-- Actuator Limits -->
   <!--  (In radians)   -->
-  <xacro:property name="actuator_pos_min" value="-1.5708"/>
-  <xacro:property name="actuator_pos_max" value="1.5708"/>
+  <xacro:property name="actuator_pos_min" value="${-pi/2}"/>
+  <xacro:property name="actuator_pos_max" value="${pi/2}"/>
+  <!-- Simulation design limits, not measured physical actuator specifications. -->
+  <xacro:property name="actuator_velocity_limit" value="10.0"/>
+  <xacro:property name="actuator_effort_limit" value="10.0"/>
+  <xacro:property name="wheel_velocity_limit" value="30.0"/>
+  <xacro:property name="wheel_effort_limit" value="10.0"/>
   <!-- Material & Visual Properties -->
   <xacro:property name="wheel_color" value="0.1 0.1 0.1 1.0"/>

File: src/swervebot_description/description/swervebot_ros2_control.xacro (robot description, xacro)
@@ -3,5 +3,5 @@
     <!-- Include the properties file to access the defined properties -->
     <xacro:include filename="$(find swervebot_description)/description/swervebot_properties.xacro" />
-    <xacro:macro name="robot_control" params="use_mock_hardware use_sim">
+    <xacro:macro name="robot_control" params="use_mock_hardware use_sim controller_config">
         <ros2_control name="SwerveBotSystem" type="system">
             <!-- Mock Hardware -->
@@ -95,9 +95,30 @@
             </joint>
         </ros2_control>
+        <!-- Model poses are diagnostics, never a second publisher of odom -> base TF. -->
+        <xacro:if value="${use_sim}">
+            <gazebo>
+                <plugin filename="gz-sim-pose-publisher-system" name="gz::sim::systems::PosePublisher">
+                    <!-- Fix the topic explicitly; URDF conversion may change scoped names. -->
+                    <topic>/model/swervebot/pose</topic>
+                    <publish_link_pose>false</publish_link_pose>
+                    <publish_sensor_pose>false</publish_sensor_pose>
+                    <publish_collision_pose>false</publish_collision_pose>
+                    <publish_visual_pose>false</publish_visual_pose>
+                    <publish_model_pose>true</publish_model_pose>
+                    <publish_nested_model_pose>false</publish_nested_model_pose>
+                    <use_pose_vector_msg>true</use_pose_vector_msg>
+                    <update_frequency>50</update_frequency>
+                </plugin>
+            </gazebo>
+        </xacro:if>
         <!-- Gazebo ROS 2 Control Plugin -->
         <xacro:if value="${use_sim}">
             <gazebo>
-                <plugin filename="libgz_ros2_control-system.so" name="gz_ros2_control::GazeboSimControl">
-                    <parameters>$(find swervebot_controllers)/config/controllers.yaml</parameters>
+                <plugin filename="libgz_ros2_control-system.so" name="gz_ros2_control::GazeboSimROS2ControlPlugin">
+                    <parameters>${controller_config}</parameters>
+                    <controller_manager_name>controller_manager</controller_manager_name>
+                    <hardware_init_timeout>30.0</hardware_init_timeout>
+                    <!-- Gain maps position error to joint velocity at the controller rate. -->
+                    <position_proportional_gain>0.1</position_proportional_gain>
                 </plugin>
             </gazebo>

File: src/swervebot_description/description/swervebot_wheel.xacro (robot description, xacro)
@@ -8,6 +8,8 @@
             <parent link="${parent_link}" />
             <child link="${name}" />
-            <origin xyz="${x} ${y} ${z}" rpy="${pi/2} 0 0" />
+            <origin xyz="${x} ${y} ${z}" rpy="${-pi/2} 0 0" />
+            <!-- Rotate local +z onto body +y: positive wheel rotation rolls body +x. -->
             <axis xyz="0 0 1" />
+            <limit effort="${wheel_effort_limit}" velocity="${wheel_velocity_limit}"/>
         </joint>
         <link name="${name}">
