Commit message: Add swerve_drive_controller as a git submodule

File: src/swervebot_description/description/swervebot.urdf.xacro (robot description, xacro)
@@ -1,15 +1,20 @@
 <?xml version="1.0"?>
 <robot xmlns:xacro="http://www.ros.org/wiki/xacro" name="swervebot">
-    <!-- Include subsystem files -->
+    <!-- Load configuration once before defining components. -->
+    <xacro:include filename="$(find swervebot_description)/description/inertia.xacro" />
     <xacro:include filename="$(find swervebot_description)/description/swervebot_properties.xacro" />
     <xacro:include filename="$(find swervebot_description)/description/swervebot_base.xacro" />
     <xacro:include filename="$(find swervebot_description)/description/swervebot_module.xacro"/>
     <xacro:include filename="$(find swervebot_description)/description/swervebot_ros2_control.xacro"/>
+    <xacro:include filename="$(find swervebot_description)/description/swervebot_lidar.xacro"/>
     <xacro:arg name="use_sim" default="false"/>
     <xacro:arg name="use_mock_hardware" default="false"/>
-    <xacro:arg name="controller_config" default="$(find swervebot_controllers)/config/controllers.yaml"/>
+    <xacro:arg name="controller_config" default="$(find swerve_drive_controller)/config/controllers.yaml"/>
     <!-- Execute/Instantiate the macros -->
     <xacro:swervebot_base />
     <xacro:add_all_swerve_modules/>
+    <xacro:if value="${lidar_enabled}">
+        <xacro:swervebot_lidar use_sim="$(arg use_sim)" />
+    </xacro:if>
     <xacro:robot_control
         use_mock_hardware="$(arg use_mock_hardware)"

File: src/swervebot_description/description/swervebot_actuator.xacro (robot description, xacro)
@@ -1,8 +1,6 @@
 <?xml version="1.0"?>
 <robot xmlns:xacro="http://www.ros.org/wiki/xacro">
-    <!-- Include the properties file to access the defined properties -->
-    <xacro:include filename="$(find swervebot_description)/description/swervebot_properties.xacro" />
-    <xacro:include filename="$(find swervebot_description)/description/inertia.xacro" />
-    <xacro:macro name="swervebot_actuator" params="name x y z parent_link">
+    <!-- Configuration and inertia helpers are loaded by the assembly entrypoint. -->
+    <xacro:macro name="swervebot_actuator" params="name x y z parent_link radius:=${actuator_radius} height:=${actuator_height} mass:=${actuator_mass}">
         <joint name="${name}_joint" type="revolute">
             <parent link="${parent_link}" />
@@ -18,5 +16,5 @@
                 <origin xyz="0 0 0" rpy="0 0 0" />
                 <geometry>
-                    <cylinder radius="${actuator_radius}" length="${actuator_height}" />
+                    <cylinder radius="${radius}" length="${height}" />
                 </geometry>
                 <material name="actuator_material">
@@ -27,11 +25,11 @@
                 <origin xyz="0 0 0" rpy="0 0 0" />
                 <geometry>
-                    <cylinder radius="${actuator_radius}" length="${actuator_height}" />
+                    <cylinder radius="${radius}" length="${height}" />
                 </geometry>
             </collision>
             <inertial>
                 <origin xyz="0 0 0" rpy="0 0 0" />
-                <mass value="${actuator_mass}" />
-                <xacro:cylinder_inertia_values m="${actuator_mass}" r="${actuator_radius}" h="${actuator_height}" />
+                <mass value="${mass}" />
+                <xacro:cylinder_inertia_values m="${mass}" r="${radius}" h="${height}" />
             </inertial>
         </link>

File: src/swervebot_description/description/swervebot_base.xacro (robot description, xacro)
@@ -1,8 +1,6 @@
 <?xml version="1.0"?>
 <robot xmlns:xacro="http://www.ros.org/wiki/xacro">
-    <!-- Include the properties file to access the defined properties -->
-    <xacro:include filename="$(find swervebot_description)/description/swervebot_properties.xacro" />
-    <xacro:include filename="$(find swervebot_description)/description/inertia.xacro" />
-    <xacro:macro name="swervebot_base" >
+    <!-- Configuration and inertia helpers are loaded by the assembly entrypoint. -->
+    <xacro:macro name="swervebot_base" params="length:=${chassis_length} width:=${chassis_width} height:=${chassis_height} mass:=${chassis_mass}" >
         <link name="base_footprint" />
         <joint name="base_footprint_joint" type="fixed">
@@ -21,5 +19,5 @@
                 <origin xyz="0 0 0" rpy="0 0 0" />
                 <geometry>
-                    <box size="${chassis_length} ${chassis_width} ${chassis_height}" />
+                    <box size="${length} ${width} ${height}" />
                 </geometry>
                 <material name="chassis_material">
@@ -30,11 +28,11 @@
                 <origin xyz="0 0 0" rpy="0 0 0" />
                 <geometry>
-                    <box size="${chassis_length} ${chassis_width} ${chassis_height}" />
+                    <box size="${length} ${width} ${height}" />
                 </geometry>
             </collision>
             <inertial>
                 <origin xyz="0 0 0" rpy="0 0 0" />
-                <mass value="${chassis_mass}" />
-                <xacro:box_inertia_values m="${chassis_mass}" x="${chassis_length}" y="${chassis_width}" z="${chassis_height}" />
+                <mass value="${mass}" />
+                <xacro:box_inertia_values m="${mass}" x="${length}" y="${width}" z="${height}" />
             </inertial>
         </link>

File: src/swervebot_description/description/swervebot_lidar.xacro (robot description, xacro)
@@ -1,49 +1,50 @@
 <?xml version="1.0"?>
 <robot xmlns:xacro="http://www.ros.org/wiki/xacro">
-    <!-- Include the properties file to access the defined properties -->
-    <xacro:include filename="$(find swervebot_description)/description/swervebot_properties.xacro" />
-    <xacro:include filename="$(find swervebot_description)/description/inertia.xacro" />
-    <link name="laser_frame">
-        <visual>
-            <geometry><cylinder radius="${lidar_radius}" length="${lidar_height}"/></geometry>
-            <material name="${lidar_color}"/>
-        </visual>
-        <collision>
-            <geometry><cylinder radius="${lidar_radius}" length="${lidar_height}"/></geometry>
-        </collision>
-    </link>
-    <joint name="laser_joint" type="fixed">
-        <parent link="base_link"/>
-        <child link="laser_frame"/>
-        <origin xyz="${lidar_x} ${lidar_y} ${lidar_z}" rpy="0 0 0"/>
-    </joint>
-    <!-- Gazebo-specific configurations for ray tracing -->
-    <gazebo reference="laser_frame">
-        <sensor name="rplidar_c1" type="gpu_lidar">
-            <pose>0 0 0 0 0 0</pose>
-            <visualize>true</visualize>
-            <update_rate>10</update_rate>
-            <ray>
-            <scan>
-                <horizontal>
-                <samples>${lidar_samples}</samples>
-                <resolution>${lidar_angle_res}</resolution>
-                <min_angle>-${lidar_min_angle}</min_angle>
-                <max_angle>${lidar_max_angle}</max_angle>
-                </horizontal>
-            </scan>
-            <range>
-                <min>${lidar_min_range}</min>
-                <max>${lidar_max_range}</max>
-                <resolution>${lidar_range_res}</resolution>
-            </range>
-            </ray>
-            <plugin filename="libgz-sim-sensors-system.so" name="gz::sim::systems::Sensors">
-            <ros>
-                <namespace>/</namespace>
-                <remapping>~/out:=scan</remapping>
-            </ros>
-            </plugin>
-        </sensor>
-    </gazebo>
+    <!-- Mount pose is parent-relative; base_link is at the chassis center. -->
+    <xacro:macro name="swervebot_lidar" params="use_sim parent_link:=${lidar_parent} xyz:='${lidar_x} ${lidar_y} ${lidar_z}' rpy:=${lidar_rpy} radius:=${lidar_radius} height:=${lidar_height} mass:=${lidar_mass}">
+        <link name="laser_frame">
+            <visual>
+                <geometry><cylinder radius="${radius}" length="${height}"/></geometry>
+                <material name="lidar_material"><color rgba="${lidar_color}"/></material>
+            </visual>
+            <collision>
+                <geometry><cylinder radius="${radius}" length="${height}"/></geometry>
+            </collision>
+            <inertial>
+                <mass value="${mass}"/>
+                <xacro:cylinder_inertia_values m="${mass}" r="${radius}" h="${height}"/>
+            </inertial>
+        </link>
+        <joint name="laser_joint" type="fixed">
+            <parent link="${parent_link}"/>
+            <child link="laser_frame"/>
+            <origin xyz="${xyz}" rpy="${rpy}"/>
+        </joint>
+        <xacro:if value="${use_sim}">
+            <gazebo reference="laser_frame">
+                <sensor name="rplidar_c1" type="gpu_lidar">
+                    <topic>${lidar_topic}</topic>
+                    <!-- Keep the ROS frame stable after Gazebo fixed-joint reduction. -->
+                    <gz_frame_id>laser_frame</gz_frame_id>
+                    <visualize>true</visualize>
+                    <update_rate>${lidar_update_rate}</update_rate>
+                    <ray>
+                        <scan>
+                            <horizontal>
+                                <samples>${lidar_samples}</samples>
+                                <resolution>${lidar_angle_res}</resolution>
+                                <min_angle>${lidar_min_angle}</min_angle>
+                                <max_angle>${lidar_max_angle}</max_angle>
+                            </horizontal>
+                        </scan>
+                        <range>
+                            <min>${lidar_min_range}</min>
+                            <max>${lidar_max_range}</max>
+                            <resolution>${lidar_range_res}</resolution>
+                        </range>
+                    </ray>
+                </sensor>
+            </gazebo>
+        </xacro:if>
+    </xacro:macro>
 </robot>

File: src/swervebot_description/description/swervebot_module.xacro (robot description, xacro)
@@ -2,5 +2,4 @@
 <robot xmlns:xacro="http://www.ros.org/wiki/xacro">
     <!-- Include subsystem files -->
-    <xacro:include filename="$(find swervebot_description)/description/swervebot_properties.xacro" />
     <xacro:include filename="$(find swervebot_description)/description/swervebot_wheel.xacro" />
     <xacro:include filename="$(find swervebot_description)/description/swervebot_actuator.xacro" />
@@ -8,5 +7,5 @@
     <!--          Create One Swerve Module            -->
     <!-- ============================================ -->
-    <xacro:macro name="add_swerve_module" params="name actuator_x actuator_y actuator_z wheel_x wheel_y wheel_z">
+    <xacro:macro name="add_swerve_module" params="name actuator_x actuator_y actuator_z wheel_x wheel_y wheel_z parent_link:=chassis">
         <xacro:swervebot_actuator
             name="actuator_${name}"
@@ -14,5 +13,5 @@
             y="${actuator_y}"
             z="${actuator_z}"
-            parent_link="chassis" />
+            parent_link="${parent_link}" />
         <xacro:swervebot_wheel
             name="wheel_${name}"
@@ -32,37 +31,37 @@
         <xacro:add_swerve_module
             name="${module_1}"
-            actuator_x="${wheelbase / 2}"
-            actuator_y="${track_width / 2}"
-            actuator_z="${actuator_offset_z}"
-            wheel_x="${wheel_offset_x}"
-            wheel_y="${wheel_offset_y}"
-            wheel_z="${wheel_offset_z}"/>
+            actuator_x="${module_1_x}"
+            actuator_y="${module_1_y}"
+            actuator_z="${module_1_z}"
+            wheel_x="${module_1_wheel_x}"
+            wheel_y="${module_1_wheel_y}"
+            wheel_z="${module_1_wheel_z}"/>
         <!-- Front Right -->
         <xacro:add_swerve_module
             name="${module_2}"
-            actuator_x="${wheelbase / 2}"
-            actuator_y="${-track_width / 2}"
-            actuator_z="${actuator_offset_z}"
-            wheel_x="${wheel_offset_x}"
-            wheel_y="${-wheel_offset_y}"
-            wheel_z="${wheel_offset_z}"/>
+            actuator_x="${module_2_x}"
+            actuator_y="${module_2_y}"
+            actuator_z="${module_2_z}"
+            wheel_x="${module_2_wheel_x}"
+            wheel_y="${module_2_wheel_y}"
+            wheel_z="${module_2_wheel_z}"/>
         <!-- Back Left -->
         <xacro:add_swerve_module
             name="${module_3}"
-            actuator_x="${-wheelbase / 2}"
-            actuator_y="${track_width / 2}"
-            actuator_z="${actuator_offset_z}"
-            wheel_x="${-wheel_offset_x}"
-            wheel_y="${wheel_offset_y}"
-            wheel_z="${wheel_offset_z}"/>
+            actuator_x="${module_3_x}"
+            actuator_y="${module_3_y}"
+            actuator_z="${module_3_z}"
+            wheel_x="${module_3_wheel_x}"
+            wheel_y="${module_3_wheel_y}"
+            wheel_z="${module_3_wheel_z}"/>
         <!-- Back Right -->
         <xacro:add_swerve_module
             name="${module_4}"
-            actuator_x="${-wheelbase / 2}"
-            actuator_y="${-track_width / 2}"
-            actuator_z="${actuator_offset_z}"
-            wheel_x="${-wheel_offset_x}"
-            wheel_y="${-wheel_offset_y}"
-            wheel_z="${wheel_offset_z}"/>
+            actuator_x="${module_4_x}"
+            actuator_y="${module_4_y}"
+            actuator_z="${module_4_z}"
+            wheel_x="${module_4_wheel_x}"
+            wheel_y="${module_4_wheel_y}"
+            wheel_z="${module_4_wheel_z}"/>
     </xacro:macro>
 </robot>

File: src/swervebot_description/description/swervebot_properties.xacro (robot description, xacro)
@@ -28,5 +28,10 @@
   <!-- Chassis Ground Clearance -->
   <xacro:property name="chassis_ground_clearance" value="${wheel_radius - actuator_offset_z - wheel_offset_z - chassis_height/2}" />
-  <!-- Lidar Properties -->
+  <!-- Lidar Properties: model in all modes, sensor only in simulation. -->
+  <xacro:property name="lidar_enabled" value="true"/>
+  <xacro:property name="lidar_parent" value="base_link"/>
+  <xacro:property name="lidar_rpy" value="0 0 0"/>
+  <xacro:property name="lidar_topic" value="/scan"/>
+  <xacro:property name="lidar_update_rate" value="10"/>
   <xacro:property name="lidar_radius" value="0.03"/>
   <xacro:property name="lidar_height" value="0.04"/>
@@ -34,13 +39,13 @@
   <xacro:property name="lidar_samples" value="500"/>
   <xacro:property name="lidar_angle_res" value="1"/>
-  <xacro:property name="lidar_min_angle" value="-3.14159"/>
-  <xacro:property name="lidar_max_angle" value="3.14159"/>
+  <xacro:property name="lidar_min_angle" value="${-pi}"/>
+  <xacro:property name="lidar_max_angle" value="${pi}"/>
   <xacro:property name="lidar_min_range" value="0.05"/>
   <xacro:property name="lidar_max_range" value="12.0"/>
   <xacro:property name="lidar_range_res" value="0.01"/>
   <!-- Lidar Position -->
-  <xacro:property name="lidar_x" value="0.15"/>
+  <xacro:property name="lidar_x" value="0.1"/>
   <xacro:property name="lidar_y" value="0.0"/>
-  <xacro:property name="lidar_z" value="${chassis_ground_clearance + chassis_height + (lidar_height / 2)}"/>
+  <xacro:property name="lidar_z" value="${chassis_height / 2 + lidar_height / 2}"/>
   <!--   ~ LIMITS ~    -->
   <!-- Actuator Limits -->
@@ -66,3 +71,28 @@
   <xacro:property name="module_3" value="back_left"/>
   <xacro:property name="module_4" value="back_right"/>
+  <!-- Per-module placement: chassis-relative pivots and steering-relative wheels. -->
+  <xacro:property name="module_1_x" value="${1 * wheelbase / 2}"/>
+  <xacro:property name="module_1_y" value="${1 * track_width / 2}"/>
+  <xacro:property name="module_1_z" value="${actuator_offset_z}"/>
+  <xacro:property name="module_1_wheel_x" value="${1 * wheel_offset_x}"/>
+  <xacro:property name="module_1_wheel_y" value="${1 * wheel_offset_y}"/>
+  <xacro:property name="module_1_wheel_z" value="${wheel_offset_z}"/>
+  <xacro:property name="module_2_x" value="${1 * wheelbase / 2}"/>
+  <xacro:property name="module_2_y" value="${-1 * track_width / 2}"/>
+  <xacro:property name="module_2_z" value="${actuator_offset_z}"/>
+  <xacro:property name="module_2_wheel_x" value="${1 * wheel_offset_x}"/>
+  <xacro:property name="module_2_wheel_y" value="${-1 * wheel_offset_y}"/>
+  <xacro:property name="module_2_wheel_z" value="${wheel_offset_z}"/>
+  <xacro:property name="module_3_x" value="${-1 * wheelbase / 2}"/>
+  <xacro:property name="module_3_y" value="${1 * track_width / 2}"/>
+  <xacro:property name="module_3_z" value="${actuator_offset_z}"/>
+  <xacro:property name="module_3_wheel_x" value="${-1 * wheel_offset_x}"/>
+  <xacro:property name="module_3_wheel_y" value="${1 * wheel_offset_y}"/>
+  <xacro:property name="module_3_wheel_z" value="${wheel_offset_z}"/>
+  <xacro:property name="module_4_x" value="${-1 * wheelbase / 2}"/>
+  <xacro:property name="module_4_y" value="${-1 * track_width / 2}"/>
+  <xacro:property name="module_4_z" value="${actuator_offset_z}"/>
+  <xacro:property name="module_4_wheel_x" value="${-1 * wheel_offset_x}"/>
+  <xacro:property name="module_4_wheel_y" value="${-1 * wheel_offset_y}"/>
+  <xacro:property name="module_4_wheel_z" value="${wheel_offset_z}"/>
 </robot>

File: src/swervebot_description/description/swervebot_ros2_control.xacro (robot description, xacro)
@@ -1,7 +1,26 @@
 <?xml version="1.0"?>
 <robot xmlns:xacro="http://www.ros.org/wiki/xacro">
-    <!-- Include the properties file to access the defined properties -->
-    <xacro:include filename="$(find swervebot_description)/description/swervebot_properties.xacro" />
+    <!-- Configuration and inertia helpers are loaded by the assembly entrypoint. -->
+    <!-- One steering position interface and one drive velocity interface per module. -->
+    <xacro:macro name="module_control" params="name">
+        <joint name="actuator_${name}_joint">
+            <command_interface name="position">
+                <param name="min">${actuator_pos_min}</param>
+                <param name="max">${actuator_pos_max}</param>
+            </command_interface>
+            <state_interface name="position"/>
+            <state_interface name="velocity"/>
+        </joint>
+        <joint name="wheel_${name}_joint">
+            <command_interface name="velocity"/>
+            <state_interface name="position"/>
+            <state_interface name="velocity"/>
+        </joint>
+    </xacro:macro>
     <xacro:macro name="robot_control" params="use_mock_hardware use_sim controller_config">
+        <!-- Fail during expansion rather than emit two competing hardware implementations. -->
+        <xacro:if value="${use_mock_hardware and use_sim}">
+            <xacro:property name="invalid_hardware" value="${xacro.fatal('use_mock_hardware and use_sim are mutually exclusive')}" lazy_eval="false"/>
+        </xacro:if>
         <ros2_control name="SwerveBotSystem" type="system">
             <!-- Mock Hardware -->
@@ -26,72 +45,8 @@
                 </hardware>
             </xacro:unless>
-            <!-- ============================================ -->
-            <!--             Module 1: Steering               -->
-            <!-- ============================================ -->
-            <joint name="actuator_${module_1}_joint">
-                <command_interface name="position">
-                    <param name="min">${actuator_pos_min}</param>
-                    <param name="max">${actuator_pos_max}</param>
-                </command_interface>
-                <state_interface name="position"/>
-                <state_interface name="velocity"/>
-            </joint>
-            <!-- Module 1: Drive Wheel -->
-            <joint name="wheel_${module_1}_joint">
-                <command_interface name="velocity"/>
-                <state_interface name="position"/>
-                <state_interface name="velocity"/>
-            </joint>
-            <!-- ============================================ -->
-            <!--             Module 2: Steering               -->
-            <!-- ============================================ -->
-            <joint name="actuator_${module_2}_joint">
-                <command_interface name="position">
-                    <param name="min">${actuator_pos_min}</param>
-                    <param name="max">${actuator_pos_max}</param>
-                </command_interface>
-                <state_interface name="position"/>
-                <state_interface name="velocity"/>
-            </joint>
-            <!-- Module 2: Drive Wheel -->
-            <joint name="wheel_${module_2}_joint">
-                <command_interface name="velocity"/>
-                <state_interface name="position"/>
-                <state_interface name="velocity"/>
-            </joint>
-            <!-- ============================================ -->
-            <!--             Module 3: Steering               -->
-            <!-- ============================================ -->
-            <joint name="actuator_${module_3}_joint">
-                <command_interface name="position">
-                    <param name="min">${actuator_pos_min}</param>
-                    <param name="max">${actuator_pos_max}</param>
-                </command_interface>
-                <state_interface name="position"/>
-                <state_interface name="velocity"/>
-            </joint>
-            <!-- Module 3: Drive Wheel -->
-            <joint name="wheel_${module_3}_joint">
-                <command_interface name="velocity"/>
-                <state_interface name="position"/>
-                <state_interface name="velocity"/>
-            </joint>
-            <!-- ============================================ -->
-            <!--             Module 4: Steering               -->
-            <!-- ============================================ -->
-            <joint name="actuator_${module_4}_joint">
-                <command_interface name="position">
-                    <param name="min">${actuator_pos_min}</param>
-                    <param name="max">${actuator_pos_max}</param>
-                </command_interface>
-                <state_interface name="position"/>
-                <state_interface name="velocity"/>
-            </joint>
-            <!-- Module 4: Drive Wheel -->
-            <joint name="wheel_${module_4}_joint">
-                <command_interface name="velocity"/>
-                <state_interface name="position"/>
-                <state_interface name="velocity"/>
-            </joint>
+            <xacro:module_control name="${module_1}"/>
+            <xacro:module_control name="${module_2}"/>
+            <xacro:module_control name="${module_3}"/>
+            <xacro:module_control name="${module_4}"/>
         </ros2_control>
         <!-- Model poses are diagnostics, never a second publisher of odom -> base TF. -->
