Commit message: Add swerve_drive_controller as a git submodule

File: src/swervebot_description/description/swervebot_wheel.xacro (robot description, xacro)
@@ -1,8 +1,6 @@
 <?xml version="1.0"?>
 <robot xmlns:xacro="http://www.ros.org/wiki/xacro">
-    <!-- Include the properties file to access the defined properties -->
-    <xacro:include filename="$(find swervebot_description)/description/swervebot_properties.xacro" />
-    <xacro:include filename="$(find swervebot_description)/description/inertia.xacro" />
-    <xacro:macro name="swervebot_wheel" params="name x y z parent_link">
+    <!-- Configuration and inertia helpers are loaded by the assembly entrypoint. -->
+    <xacro:macro name="swervebot_wheel" params="name x y z parent_link radius:=${wheel_radius} width:=${wheel_width} mass:=${wheel_mass}">
         <joint name="${name}_joint" type="continuous">
             <parent link="${parent_link}" />
@@ -17,5 +15,5 @@
                 <origin xyz="0 0 0" rpy="0 0 0" />
                 <geometry>
-                    <cylinder radius="${wheel_radius}" length="${wheel_width}" />
+                    <cylinder radius="${radius}" length="${width}" />
                 </geometry>
                 <material name="wheel_material">
@@ -26,11 +24,11 @@
                 <origin xyz="0 0 0" rpy="0 0 0" />
                 <geometry>
-                    <cylinder radius="${wheel_radius}" length="${wheel_width}" />
+                    <cylinder radius="${radius}" length="${width}" />
                 </geometry>
             </collision>
             <inertial>
                 <origin xyz="0 0 0" rpy="0 0 0" />
-                <mass value="${wheel_mass}" />
-                <xacro:cylinder_inertia_values m="${wheel_mass}" r="${wheel_radius}" h="${wheel_width}" />
+                <mass value="${mass}" />
+                <xacro:cylinder_inertia_values m="${mass}" r="${radius}" h="${width}" />
             </inertial>
         </link>
